Commit message: tweaked inertia

File: tbd_podi_description/urdf/inertia_tensors.xacro (robot description, xacro)
@@ -5,5 +5,5 @@
   see http://answers.gazebosim.org/question/4372/the-inertia-matrix-explained/ -->
 <robot xmlns:xacro="http://ros.org/wiki/xacro">
-  <property name="M_PI" value="3.1415926535897931" />
+  <xacro:property name="M_PI" value="3.1415926535897931" />
   <!-- see https://secure.wikimedia.org/wikipedia/en/wiki/List_of_moment_of_inertia_tensors -->
   <!-- #################### versions without origin #################### -->
@@ -26,4 +26,13 @@
     </inertial>
   </xacro:macro>
+  <xacro:macro name="hollow_cylinder_inertial" params="radius inner_radius length mass">
+    <inertial>
+      <mass value="${mass}" />
+      <origin xyz="0 0 0" />
+      <inertia ixx="${0.0833333 * mass * (3 * (radius * radius + inner_radius * inner_radius) + length * length)}" ixy="0.0" ixz="0.0"
+        iyy="${0.0833333 * mass * (3 * (radius * radius + inner_radius * inner_radius) + length * length)}" iyz="0.0"
+        izz="${0.5 * mass * (radius * radius + inner_radius * inner_radius)}" />
+    </inertial>
+  </xacro:macro>
   <xacro:macro name="box_inertial" params="x y z mass">
     <inertial>
@@ -39,5 +48,5 @@
     <inertial>
       <mass value="${mass}" />
-      <insert_block name="origin" />
+      <xacro:insert_block name="origin" />
       <inertia ixx="${0.4 * mass * radius * radius}" ixy="0.0" ixz="0.0"
         iyy="${0.4 * mass * radius * radius}" iyz="0.0"
@@ -48,5 +57,5 @@
     <inertial>
       <mass value="${mass}" />
-      <insert_block name="origin" />
+      <xacro:insert_block name="origin" />
       <inertia ixx="${0.0833333 * mass * (3 * radius * radius + length * length)}" ixy="0.0" ixz="0.0"
         iyy="${0.0833333 * mass * (3 * radius * radius + length * length)}" iyz="0.0"
@@ -54,8 +63,17 @@
     </inertial>
   </xacro:macro>
+  <xacro:macro name="hollow_cylinder_inertial_with_origin" params="radius inner_radius length mass *origin">
+    <inertial>
+      <mass value="${mass}" />
+      <xacro:insert_block name="origin" />
+      <inertia ixx="${0.0833333 * mass * (3 * (radius * radius + inner_radius * inner_radius) + length * length)}" ixy="0.0" ixz="0.0"
+        iyy="${0.0833333 * mass * (3 * (radius * radius + inner_radius * inner_radius) + length * length)}" iyz="0.0"
+        izz="${0.5 * mass * (radius * radius + inner_radius * inner_radius)}" />
+    </inertial>
+  </xacro:macro>
   <xacro:macro name="box_inertial_with_origin" params="x y z mass *origin">
     <inertial>
       <mass value="${mass}" />
-      <insert_block name="origin" />
+      <xacro:insert_block name="origin" />
       <inertia ixx="${0.0833333 * mass * (y*y + z*z)}" ixy="0.0" ixz="0.0"
         iyy="${0.0833333 * mass * (x*x + z*z)}" iyz="0.0"

File: tbd_podi_description/urdf/pioneer3dx.urdf.xacro (robot description, xacro)
@@ -26,9 +26,5 @@
     </gazebo>
     <link name="top_plate">
-        <inertial>
-            <mass value="0.01"/>
-            <origin xyz="0 0 0"/>
-            <inertia ixx="1" ixy="0" ixz="0" iyy="1" iyz="0" izz="1"/>
-        </inertial>
+        <xacro:box_inertial x="0.45" y="0.38" z="0.01" mass="0.5" />
         <visual>
             <origin xyz="0 0 0" rpy="0 0 0"/>
@@ -118,5 +114,5 @@
     <link name="caster_swivel">
         <inertial>
-            <mass value="0.1"/>
+            <mass value="0.01"/>
             <origin xyz="0 0 0"/>
             <inertia ixx="0.01" ixy="0" ixz="0" iyy="0.01" iyz="0" izz="0.01"/>
@@ -145,9 +141,5 @@
     </joint>
     <link name="caster_wheel">
-        <inertial>
-            <mass value="0.1"/>
-            <origin xyz="0 0 0"/>
-            <inertia ixx="0.012411765597" ixy="-0.000711733678" ixz="0.00050272983" iyy="0.015218160428" iyz="-0.000004273467" izz="0.011763977943"/>
-        </inertial>
+        <xacro:cylinder_inertial radius="0.0375" length="0.01" mass="0.5" />
         <visual>
             <origin xyz="0 0 0" rpy="0 0 0"/>

File: tbd_podi_description/urdf/pioneer3dx_wheel.xacro (robot description, xacro)
@@ -4,11 +4,9 @@
   <xacro:macro name="p3dx_wheel" params="suffix reflect parent">
     <link name="${suffix}_wheel">
-      <inertial>
-        <mass value="0.5"/>
-        <origin xyz="0 0 0"/>
-        <inertia ixx="0.012411765597" ixy="0" ixz="0" iyy="0.015218160428" iyz="0" izz="0.011763977943"/>
-      </inertial>
+      <xacro:hollow_cylinder_inertial radius="0.09" inner_radius="0.05" length="0.04" mass="1" />
       <visual>
         <origin xyz="0 0 0" rpy="0 0 0"/>
+        <!-- The wheel isn't a perfect cylinder. -->
+        <!-- Radius: 0.09, inner radius:0.05, length:0.04 -->
         <geometry name="pioneer_geom">
           <mesh filename="package://tbd_podi_description/meshes/p3dx_meshes/${suffix}_wheel.stl"/>
@@ -21,5 +19,5 @@
         <origin xyz="0 0 0" rpy="${-3.1415927/2} 0 0"/>
         <geometry>
-          <cylinder radius="0.09" length="0.01"/>
+          <cylinder radius="0.09" length="0.04"/>
         </geometry>
       </collision>
@@ -32,6 +30,7 @@
     </joint>
     <link name="${suffix}_hubcap">
+      <!-- It's a big hard to model the exact inertia, so let's ignore it here. -->
       <inertial>
-        <mass value="0.01"/>
+        <mass value="0.00"/>
         <origin xyz="0 0 0"/>
         <inertia ixx="0.012411765597" ixy="0" ixz="0" iyy="0.015218160428" iyz="0" izz="0.011763977943"/>
@@ -39,4 +38,5 @@
       <visual>
         <origin xyz="0 0 0" rpy="0 0 0"/>
+        <!-- It is actually two disk shape object on both side of the wheel -->
         <geometry name="pioneer_geom">
           <mesh filename="package://tbd_podi_description/meshes/p3dx_meshes/${suffix}_hubcap.stl"/>
@@ -49,5 +49,5 @@
         <origin xyz="0 0 0" rpy="0 0 0"/>
         <geometry>
-          <box size="0 0 0"/>
+          <cylinder radius="0.05" length="0.03"/>
         </geometry>
       </collision>

File: tbd_podi_description/urdf/podi.gazebo.xacro (robot description, xacro)
@@ -12,5 +12,5 @@
       <publishWheelJointState>true</publishWheelJointState>
       <publishWheelTF>false</publishWheelTF>
-      <wheelAcceleration>1.8</wheelAcceleration>
+      <wheelAcceleration>1</wheelAcceleration>
       <commandTopic>cmd_vel</commandTopic>
       <odometryTopic>odom</odometryTopic>

File: tbd_podi_description/urdf/podi_handle.xacro (robot description, xacro)
@@ -20,9 +20,5 @@
     </link>
     <link name="handle_bottom_plate">
-        <inertial>
-            <mass value="1" />
-            <origin xyz="0 0 0" />
-            <inertia ixx="1" ixy="0" ixz="0" iyy="1" iyz="0" izz="1" />
-        </inertial>
+        <xacro:box_inertial x="0.09" y="0.21" z="0.005" mass="1" />
         <visual>
             <origin xyz="0 0 0" rpy="0 0 0"/>

File: tbd_podi_description/urdf/podi_structure.xacro (robot description, xacro)
@@ -2,9 +2,5 @@
 <robot xmlns:xacro="http://ros.org/wiki/xacro">
     <link name="laser_scanner">
-        <inertial>
-            <mass value="1" />
-            <origin xyz="0 0 0" />
-            <inertia ixx="1" ixy="0" ixz="0" iyy="1" iyz="0" izz="1" />
-        </inertial>
+        <xacro:box_inertial x="0.105" y="0.102" z="0.152" mass="0.429" />
         <visual>
             <origin xyz="0 0 0" rpy="0 0 0"/>
@@ -28,13 +24,9 @@
         <child link="laser_scanner"/>
     </joint>
-    <xacro:property name="face_screen_width" value="0.01" />
-    <xacro:property name="face_screen_height" value="0.2" />
-    <xacro:property name="face_screen_length" value="0.2" />
+    <xacro:property name="face_screen_width" value="0.006" />
+    <xacro:property name="face_screen_height" value="0.2373" />
+    <xacro:property name="face_screen_length" value="0.169" />
     <link name="${robotname}_face_screen">
-        <inertial>
-            <mass value="0.5" />
-            <origin xyz="0 0 0" />
-            <inertia ixx="1" ixy="0" ixz="0" iyy="1" iyz="0" izz="1" />
-        </inertial>
+        <xacro:box_inertial x="${face_screen_width}" y="${face_screen_length}" z="${face_screen_height}" mass="0.429" />
         <visual>
             <origin xyz="0 0 0" rpy="0 0 0"/>
