Commit message: fixed namespace

File: tbd_podi_description/urdf/pioneer3dx.urdf.xacro (robot description, xacro)
@@ -4,5 +4,5 @@
     <xacro:include filename="$(find tbd_podi_description)/urdf/pioneer3dx_wheel.xacro"/>
     <!-- Chassis -->
-    <link name="base_link">
+    <link name="$(arg robot_name)_base_link">
         <xacro:box_inertial x="0.35" y="0.25" z="0.14" mass="10" />
         <visual>
@@ -22,8 +22,8 @@
         </collision>
     </link>
-    <gazebo reference="base_link">
+    <gazebo reference="$(arg robot_name)_base_link">
         <material>Gazebo/Red</material>
     </gazebo>
-    <link name="top_plate">
+    <link name="$(arg robot_name)_top_plate">
         <xacro:box_inertial x="0.45" y="0.38" z="0.01" mass="0.5" />
         <visual>
@@ -43,14 +43,14 @@
         </collision>
     </link>
-    <gazebo reference="top_plate">
+    <gazebo reference="$(arg robot_name)_top_plate">
         <material>Gazebo/Black</material>
     </gazebo>
-    <joint name="base_top_joint" type="fixed">
+    <joint name="$(arg robot_name)_base_top_joint" type="fixed">
         <origin xyz="-0.045 0 0.234" rpy="0 0 0"/>
         <axis xzy="0 0 1"/>
-        <parent link="base_link"/>
-        <child link="top_plate"/>
+        <parent link="$(arg robot_name)_base_link"/>
+        <child link="$(arg robot_name)_top_plate"/>
     </joint>
-    <link name="front_sonar">
+    <link name="$(arg robot_name)_front_sonar">
         <inertial>
             <mass value="0.0001"/>
@@ -68,18 +68,18 @@
         </visual>
     </link>
-    <gazebo reference="front_sonar">
+    <gazebo reference="$(arg robot_name)_front_sonar">
         <material value="Gazebo/Yellow"/>
     </gazebo>
-    <joint name="base_front_joint" type="fixed">
+    <joint name="$(arg robot_name)_base_front_joint" type="fixed">
         <origin xyz="-0.198 0 0.208" rpy="0 0 0"/>
-        <parent link="base_link"/>
-        <child link="front_sonar"/>
+        <parent link="$(arg robot_name)_base_link"/>
+        <child link="$(arg robot_name)_front_sonar"/>
     </joint>
-    <joint name="base_back_joint" type="fixed">
+    <joint name="$(arg robot_name)_base_back_joint" type="fixed">
         <origin xyz="0.109 0 0.209" rpy="0 0 0"/>
-        <parent link="base_link"/>
-        <child link="back_sonar"/>
+        <parent link="$(arg robot_name)_base_link"/>
+        <child link="$(arg robot_name)_back_sonar"/>
     </joint>
-    <link name="back_sonar">
+    <link name="$(arg robot_name)_back_sonar">
         <inertial>
             <mass value="0"/>
@@ -104,13 +104,13 @@
     </link>
     <!-- Caster -->
-    <joint name="base_caster_swivel_joint" type="continuous">
+    <joint name="$(arg robot_name)_base_caster_swivel_joint" type="continuous">
         <origin xyz="-0.185 0 0.055" rpy="0 0 0"/>
         <axis xyz="0 0 1"/>
         <limit effort="100" velocity="100" k_velocity="0" />
         <joint_properties damping="0.0" friction="0.0" />
-        <parent link="base_link"/>
-        <child link="caster_swivel"/>
+        <parent link="$(arg robot_name)_base_link"/>
+        <child link="$(arg robot_name)_caster_swivel"/>
     </joint>
-    <link name="caster_swivel">
+    <link name="$(arg robot_name)_caster_swivel">
         <inertial>
             <mass value="0.01"/>
@@ -123,13 +123,13 @@
                 <mesh filename="package://tbd_podi_description/meshes/p3dx_meshes/caster_swivel.stl"/>
             </geometry>
-            <material name="caster_swivel">
+            <material name="$(arg robot_name)_caster_swivel">
                 <color rgba="0.5 0.5 0.5 1"/>
             </material>
         </visual>
     </link>
-    <gazebo reference="caster_swivel">
+    <gazebo reference="$(arg robot_name)_caster_swivel">
         <material value="Gazebo/Grey"/>
     </gazebo>
-    <joint name="caster_swivel_hubcap_joint" type="continuous">
+    <joint name="$(arg robot_name)_caster_swivel_hubcap_joint" type="continuous">
         <origin xyz="-0.026 0 -0.016" rpy="0 0 0"/>
         <axis xyz="0 1 0"/>
@@ -137,8 +137,8 @@
         <limit effort="100" velocity="100" k_velocity="0" />
         <joint_properties damping="0.0" friction="0.0" />
-        <parent link="caster_swivel"/>
-        <child link="caster_wheel"/>
+        <parent link="$(arg robot_name)_caster_swivel"/>
+        <child link="$(arg robot_name)_caster_wheel"/>
     </joint>
-    <link name="caster_wheel">
+    <link name="$(arg robot_name)_caster_wheel">
         <xacro:cylinder_inertial radius="0.0375" length="0.01" mass="0.5" />
         <visual>
@@ -158,13 +158,13 @@
         </collision>
     </link>
-    <gazebo reference="caster_wheel">
+    <gazebo reference="$(arg robot_name)_caster_wheel">
         <material>Gazebo/Black</material>
     </gazebo>
-    <joint name="caster_wheel_joint" type="fixed">
+    <joint name="$(arg robot_name)_caster_wheel_joint" type="fixed">
         <origin xyz="-0.0035 0 -0.001" rpy="0 0 0"/>
-        <parent link="caster_wheel"/>
-        <child link="caster_hubcap"/>
+        <parent link="$(arg robot_name)_caster_wheel"/>
+        <child link="$(arg robot_name)_caster_hubcap"/>
     </joint>
-    <link name="caster_hubcap">
+    <link name="$(arg robot_name)_caster_hubcap">
         <inertial>
             <mass value="0.01"/>
@@ -177,5 +177,5 @@
                 <mesh filename="package://tbd_podi_description/meshes/p3dx_meshes/caster_hubcap.stl"/>
             </geometry>
-            <material name="caster_swivel">
+            <material name="$(arg robot_name)_caster_swivel">
                 <color rgba="0.5 0.5 0.5 1"/>
             </material>
@@ -188,12 +188,8 @@
         </collision>
     </link>
-    <gazebo reference="caster_hubcap">
+    <gazebo reference="$(arg robot_name)_caster_hubcap">
         <material value="Gazebo/Grey"/>
     </gazebo>
-    <xacro:p3dx_wheel suffix="left" parent="base_link" reflect="1"/>
-    <xacro:p3dx_wheel suffix="right" parent="base_link" reflect="-1"/>
-    <create>
-        <back_sonar parent="base_link"/>
-        <top_plate parent="base_link"/>
-    </create>
+    <xacro:p3dx_wheel tf_suffix="$(arg robot_name)_left" suffix="left" parent="$(arg robot_name)_base_link" reflect="1"/>
+    <xacro:p3dx_wheel tf_suffix="$(arg robot_name)_right"  suffix="right" parent="$(arg robot_name)_base_link" reflect="-1"/>
 </robot>

File: tbd_podi_description/urdf/pioneer3dx_wheel.xacro (robot description, xacro)
@@ -2,6 +2,6 @@
 <robot xmlns:xacro="http://ros.org/wiki/xacro">
   <!-- Right/Left Hubcap + Wheel -->
-  <xacro:macro name="p3dx_wheel" params="suffix reflect parent">
-    <link name="${suffix}_wheel">
+  <xacro:macro name="p3dx_wheel" params="tf_suffix suffix reflect parent">
+    <link name="${tf_suffix}_wheel">
       <xacro:hollow_cylinder_inertial radius="0.09" inner_radius="0.05" length="0.04" mass="1" />
       <visual>
@@ -23,11 +23,11 @@
       </collision>
     </link>
-    <joint name="${suffix}_hubcap_joint" type="fixed">
+    <joint name="${tf_suffix}_hubcap_joint" type="fixed">
       <!--<origin xyz="0 ${reflect*0.158} 0.091" rpy="0 0 0"/>-->
       <origin xyz="0 0 0" rpy="0 0 0"/>
-      <parent link="${suffix}_wheel"/>
-      <child link="${suffix}_hubcap"/>
+      <parent link="${tf_suffix}_wheel"/>
+      <child link="${tf_suffix}_hubcap"/>
     </joint>
-    <link name="${suffix}_hubcap">
+    <link name="${tf_suffix}_hubcap">
       <!-- It's a big hard to model the exact inertia, so let's ignore it here. -->
       <inertial>
@@ -54,27 +54,27 @@
     </link>
     <!-- Parent to the wheel -->
-    <joint name="${suffix}_wheel_joint" type="continuous">
+    <joint name="${tf_suffix}_wheel_joint" type="continuous">
       <axis xyz="0 1 0"/>
       <origin xyz="0 ${reflect*0.158} 0.091" rpy="0 0 0"/>
       <parent link="${parent}"/>
-      <child link="${suffix}_wheel"/>
+      <child link="${tf_suffix}_wheel"/>
     </joint>
     <!-- Transmission variable for gazebo -->
     <!-- This is commented out because it is used by gazebo_ros_controller, it will superseed
     the internal wheel controller if set
-    <transmission type="pr2_mechanism_model/SimpleTransmission" name="${suffix}_wheel_trans">
+    <transmission type="pr2_mechanism_model/SimpleTransmission" name="${tf_suffix}_wheel_trans">
       <type>transmission_interface/SimpleTransmission</type>
-      <actuator name="${suffix}_wheel_motor">
+      <actuator name="${tf_suffix}_wheel_motor">
         <hardwareInterface>hardware_interface/VelocityJointInterface</hardwareInterface>
         <mechanicalReduction>${reflect * 624/35 * 80/19}</mechanicalReduction>
       </actuator>
-      <joint name="${suffix}_wheel_joint">
+      <joint name="${tf_suffix}_wheel_joint">
         <hardwareInterface>hardware_interface/VelocityJointInterface</hardwareInterface>
       </joint>
     </transmission> -->
-    <gazebo reference="${suffix}_hubcap">
+    <gazebo reference="${tf_suffix}_hubcap">
       <material value="Gazebo/Yellow"/>
     </gazebo>
-    <gazebo reference="${suffix}_wheel">
+    <gazebo reference="${tf_suffix}_wheel">
       <material value="Gazebo/Black"/>
       <elem key="mu1" value="0.5" />

File: tbd_podi_description/urdf/podi.gazebo.xacro (robot description, xacro)
@@ -5,6 +5,6 @@
       <alwaysOn>true</alwaysOn>
       <updateRate>100</updateRate>
-      <leftJoint>left_wheel_joint</leftJoint>
-      <rightJoint>right_wheel_joint</rightJoint>
+      <leftJoint>$(arg robot_name)_left_wheel_joint</leftJoint>
+      <rightJoint>$(arg robot_name)_right_wheel_joint</rightJoint>
       <wheelSeparation>0.316</wheelSeparation>
       <wheelDiameter>0.18</wheelDiameter>
@@ -13,16 +13,15 @@
       <publishWheelTF>false</publishWheelTF>
       <wheelAcceleration>1</wheelAcceleration>
-      <commandTopic>cmd_vel</commandTopic>
-      <odometryTopic>odom</odometryTopic>
-      <odometryFrame>odom</odometryFrame>
-      <robotBaseFrame>base_link</robotBaseFrame>
-      <robotNamespace>${robotname}</robotNamespace>
+      <commandTopic>$(arg robot_name)/cmd_vel</commandTopic>
+      <odometryTopic>$(arg robot_name)/odom</odometryTopic>
+      <odometryFrame>$(arg robot_name)_odom</odometryFrame>
+      <robotBaseFrame>$(arg robot_name)_base_link</robotBaseFrame>
       <odometrySource>encoder</odometrySource>      <!-- The options are world and encoder. World means getting it straight from Gazebo -->
     </plugin>
     <!-- ground truth -->
-    <plugin name="p3d_base_controller" filename="libgazebo_ros_p3d.so">
+    <!-- <plugin name="p3d_base_controller" filename="libgazebo_ros_p3d.so">
       <alwaysOn>true</alwaysOn>
       <updateRate>100.0</updateRate>
-      <bodyName>base_link</bodyName>
+      <bodyName>"$(arg robot_name)_base_link"</bodyName>
       <topicName>${robotname}/pose_ground_truth</topicName>
       <gaussianNoise>0.01</gaussianNoise>
@@ -30,7 +29,7 @@
       <xyzOffsets>0 0 0</xyzOffsets>
       <rpyOffsets>0 0 0</rpyOffsets>
-    </plugin>
+    </plugin> -->
   </gazebo>
-  <gazebo reference="laser_scanner">
+  <gazebo reference="$(arg robot_name)_laser_scanner">
     <sensor type="ray" name="lms100x">
       <pose>0 0 0 0 0 0</pose>
@@ -57,12 +56,11 @@
         </noise>
       </ray>
-      <plugin name="${robotname}_front_lidar_controller" filename="libgazebo_ros_laser.so">
-        <topicName>laser</topicName>
-        <frameName>${robotname}/laser_scanner</frameName>
-        <robotNamespace>${robotname}</robotNamespace>
+      <plugin name="$(arg robot_name)_front_lidar_controller" filename="libgazebo_ros_laser.so">
+        <topicName>$(arg robot_name)/laser</topicName>
+        <frameName>$(arg robot_name)_laser_scanner</frameName>
       </plugin>
     </sensor>
   </gazebo>
-  <gazebo reference="display">
+  <gazebo reference="$(arg robot_name)_display">
     <visual>
       <plugin name="screen_video_controller" filename="libgazebo_ros_video.so">
@@ -70,9 +68,9 @@
         <width>720</width>
         <topicName>screen_face</topicName>
-        <robotNamespace>${robotname}</robotNamespace>
+        <robotNamespace>$(arg robot_name)</robotNamespace>
       </plugin>
     </visual>
   </gazebo>
-  <gazebo reference="zed_left_camera_frame">
+  <gazebo reference="$(arg robot_name)_front_camera_left_camera_frame">
     <sensor type="depth" name="front_depth_camera">
       <update_rate>30.0</update_rate>
@@ -87,5 +85,5 @@
       <plugin name="head_depth_camera" filename="libgazebo_ros_depth_camera.so">
         <cameraName>front_camera</cameraName>
-        <frameName>${robotname}/zed_left_camera_optical_frame</frameName>
+        <frameName>$(arg robot_name)_front_camera_left_camera_optical_frame</frameName>
         <robotNamespace>${robotname}</robotNamespace>
         <pointCloudCutoff>2.0</pointCloudCutoff>

File: tbd_podi_description/urdf/podi.urdf.xacro (robot description, xacro)
@@ -2,7 +2,9 @@
 <robot name="podi"
     xmlns:xacro="http://ros.org/wiki/xacro">
+    <!-- XACRO Properties and Arguments -->
+    <xacro:arg name="robot_name" default="podi" />
+    <xacro:arg name="handle_control" default="fixed" /> <!-- "fixed" if you don't want the handle to move. "move" for full rotation -->
     <xacro:property name="robotname" value="podi" />
-    <!-- "fixed" if you don't want the handle to move. "move" for full rotation -->
-    <xacro:property name="handle_control" value="fixed" />
+    <xacro:property name="handle_control" value="$(arg handle_control)" />
     <!-- Inport helper functions -->
     <xacro:include filename="$(find tbd_podi_description)/urdf/inertia_tensors.xacro"/>
@@ -12,5 +14,5 @@
     <!-- Import the handle -->
     <xacro:include filename="$(find tbd_podi_description)/urdf/podi_handle.xacro"/>
-    <!-- Import the structure -->
+    <!-- Import the top structure -->
     <xacro:include filename="$(find tbd_podi_description)/urdf/podi_structure.xacro"/>
     <!-- Gazebo -->

File: tbd_podi_description/urdf/podi_handle.xacro (robot description, xacro)
@@ -1,5 +1,5 @@
 <?xml version="1.0"?>
 <robot xmlns:xacro="http://ros.org/wiki/xacro">
-    <link name="handle_base">
+    <link name="$(arg robot_name)_handle_base">
         <xacro:cylinder_inertial radius="0.06" length="0.04" mass="10" />
         <visual>
@@ -19,5 +19,5 @@
         </collision>
     </link>
-    <link name="handle_bottom_plate">
+    <link name="$(arg robot_name)_handle_bottom_plate">
         <xacro:box_inertial x="0.09" y="0.21" z="0.005" mass="1" />
         <visual>
@@ -37,5 +37,5 @@
         </collision>
     </link>
-    <link name="handle_back_plate">
+    <link name="$(arg robot_name)_handle_back_plate">
         <inertial>
             <mass value="0.01" />
@@ -59,5 +59,5 @@
         </collision>
     </link>
-    <link name="handle_bottom">
+    <link name="$(arg robot_name)_handle_bottom">
         <inertial>
             <mass value="0.01" />
@@ -81,5 +81,5 @@
         </collision>
     </link>
-    <link name="handle_top">
+    <link name="$(arg robot_name)_handle_top">
         <inertial>
             <mass value="0.01" />
@@ -103,14 +103,14 @@
         </collision>
     </link>
-    <joint name="handle_base_joint" type="fixed">
+    <joint name="$(arg robot_name)_handle_base_joint" type="fixed">
         <origin xyz="-0.13 0 0.234" rpy="0 0 0"/>
-        <parent link="base_link"/>
-        <child link="handle_base"/>
+        <parent link="$(arg robot_name)_base_link"/>
+        <child link="$(arg robot_name)_handle_base"/>
     </joint>
-    <joint name="handle_rotation" type="revolute">
+    <joint name="$(arg robot_name)_handle_rotation" type="revolute">
         <origin xyz="0 0 0.04" rpy="0 0 0"/>
         <axis xyz = "0 0 1" />
-        <parent link="handle_base"/>
-        <child link="handle_bottom_plate"/>
+        <parent link="$(arg robot_name)_handle_base"/>
+        <child link="$(arg robot_name)_handle_bottom_plate"/>
         <xacro:if value="${handle_control == 'fixed'}">
             <limit lower="-0.01" upper="0.01" effort="1" velocity="1" />
@@ -120,19 +120,19 @@
         </xacro:if>
     </joint>
-    <joint name="handle_bottom_plate_to_back_plate" type="fixed">
+    <joint name="$(arg robot_name)_handle_bottom_plate_to_back_plate" type="fixed">
         <origin xyz="0.045 0 0.005" rpy="0 0.785398 0"/>
-        <parent link="handle_bottom_plate"/>
-        <child link="handle_back_plate"/>
+        <parent link="$(arg robot_name)_handle_bottom_plate"/>
+        <child link="$(arg robot_name)_handle_back_plate"/>
     </joint>
-    <joint name="handle_back_plate_to_bottom" type="fixed">
+    <joint name="$(arg robot_name)_handle_back_plate_to_bottom" type="fixed">
         <origin xyz="-0.14 0 0.005" rpy="0 0 0"/>
-        <parent link="handle_back_plate"/>
-        <child link="handle_bottom"/>
+        <parent link="$(arg robot_name)_handle_back_plate"/>
+        <child link="$(arg robot_name)_handle_bottom"/>
     </joint>
-    <joint name="handle_length" type="prismatic">
+    <joint name="$(arg robot_name)_handle_length" type="prismatic">
         <origin xyz="-0.33 0 0.0275" rpy="0 0 0"/>
         <axis xyz ="-1 0 0" />
-        <parent link="handle_bottom"/>
-        <child link="handle_top"/>
+        <parent link="$(arg robot_name)_handle_bottom"/>
+        <child link="$(arg robot_name)_handle_top"/>
         <limit lower="0" upper="0.46" effort="0" velocity="1" />
     </joint>

File: tbd_podi_description/urdf/podi_structure.xacro (robot description, xacro)
@@ -1,5 +1,5 @@
 <?xml version="1.0"?>
 <robot xmlns:xacro="http://ros.org/wiki/xacro">
-    <link name="laser_scanner">
+    <link name="$(arg robot_name)_laser_scanner">
         <xacro:box_inertial x="0.105" y="0.102" z="0.152" mass="0.429" />
         <visual>
@@ -19,13 +19,13 @@
         </collision>
     </link>
-    <joint name="laser_scanner_to_base_joint" type="fixed">
+    <joint name="$(arg robot_name)_laser_scanner_to_base_joint" type="fixed">
         <origin xyz="0.015 0 0.15" rpy="${pi} 0 0"/>
-        <parent link="back_sonar"/>
-        <child link="laser_scanner"/>
+        <parent link="$(arg robot_name)_back_sonar"/>
+        <child link="$(arg robot_name)_laser_scanner"/>
     </joint>
     <xacro:property name="face_screen_width" value="0.006" />
     <xacro:property name="face_screen_height" value="0.2373" />
     <xacro:property name="face_screen_length" value="0.169" />
-    <link name="face_screen">
+    <link name="$(arg robot_name)_face_screen">
         <xacro:box_inertial x="${face_screen_width}" y="${face_screen_length}" z="${face_screen_height}" mass="0.429" />
         <visual>
@@ -45,5 +45,5 @@
         </collision>
     </link>
-    <link name="head">
+    <link name="$(arg robot_name)_head">
         <inertial>
             <mass value="0.01" />
@@ -52,18 +52,18 @@
         </inertial>
     </link>
-    <joint name="head_to_screen_joint" type="fixed">
+    <joint name="$(arg robot_name)_head_to_screen_joint" type="fixed">
         <origin xyz="0 0 0" rpy="0 0 0"/>
-        <parent link="head"/>
-        <child link="face_screen"/>
+        <parent link="$(arg robot_name)_head"/>
+        <child link="$(arg robot_name)_face_screen"/>
     </joint>
-    <joint name="screen_to_laser_scanner_joint" type="fixed">
+    <joint name="screen_to_$(arg robot_name)_laser_scanner_joint" type="fixed">
         <origin xyz="0.0 0 ${0.15 + face_screen_height + 0.05}" rpy="0 0 0"/>
-        <parent link="back_sonar"/>
-        <child link="head"/>
+        <parent link="$(arg robot_name)_back_sonar"/>
+        <child link="$(arg robot_name)_head"/>
     </joint>
     <xacro:property name="display_width" value="0.01" />
     <xacro:property name="display_height" value="0.10125" />
     <xacro:property name="display_length" value="0.18" />
-    <link name="display">
+    <link name="$(arg robot_name)_display">
         <inertial>
             <mass value="0.01" />
@@ -87,23 +87,24 @@
         </collision>
     </link>
-    <joint name="display_to_screen_joint" type="fixed">
+    <joint name="$(arg robot_name)_display_to_screen_joint" type="fixed">
         <origin xyz="0.01 0 0" rpy="${3.1415927/2.0} 0 ${3.1415927/2.0}"/>
-        <parent link="face_screen"/>
-        <child link="display"/>
+        <parent link="$(arg robot_name)_face_screen"/>
+        <child link="$(arg robot_name)_display"/>
     </joint>
-   <joint name="camera_mount_to_screen_joint" type="fixed">
+   <joint name="$(arg robot_name)_camera_mount_to_screen_joint" type="fixed">
         <origin xyz="0.025 0 ${face_screen_height/2 + 0.025}" rpy="0 0 0"/>
         <axis xyz="0 1 0"/>
-        <parent link="face_screen"/>
-        <child link="front_camera_mount"/>
+        <parent link="$(arg robot_name)_face_screen"/>
+        <child link="$(arg robot_name)_front_camera_mount"/>
     </joint>
-    <xacro:arg name="base_frame" default="front_camera_mount"/>
+    <xacro:arg name="base_frame" default="$(arg robot_name)_front_camera_mount"/>
     <xacro:arg name="camera_model" default="zed2"/>
+    <xacro:arg name="camera_name" default="$(arg robot_name)_front_camera"/>
     <xacro:include filename="$(find tbd_podi_description)/urdf/zed_descr.urdf.xacro">
     </xacro:include>
     <!-- camera_name="zed2" camera_model="zed2" base_frame="${robotname_camera_mount}"/> -->
     <!-- Include Azure Kinect -->
-    <!-- <xacro:insert_azure_kinect parent="front_camera_mount" tf_prefix=""/> -->
-    <!-- <link name="front_camera_mount">
+    <!-- <xacro:insert_azure_kinect parent="$(arg robot_name)_front_camera_mount" tf_prefix=""/> -->
+    <!-- <link name="$(arg robot_name)_front_camera_mount">
         <inertial>
             <mass value="0.0001" />
