Commit message: integrating localization node

File: tbd_podi_description/urdf/pioneer3dx.urdf.xacro (robot description, xacro)
@@ -5,4 +5,6 @@
     <!-- Chassis -->
     <link name="$(arg robot_name)_base_link">
+    </link>
+    <link name="$(arg robot_name)_base_link_dummy">
         <xacro:box_inertial x="0.35" y="0.25" z="0.14" mass="10" />
         <visual>
@@ -22,7 +24,11 @@
         </collision>
     </link>
-    <gazebo reference="$(arg robot_name)_base_link">
+    <gazebo reference="$(arg robot_name)_base_link_dummy">
         <material>Gazebo/Red</material>
     </gazebo>
+    <joint name = "dummy_joint" type = "fixed">
+    	<parent link="$(arg robot_name)_base_link"/>
+    	<child link="$(arg robot_name)_base_link_dummy"/>
+    </joint>
     <link name="$(arg robot_name)_top_plate">
         <xacro:box_inertial x="0.45" y="0.38" z="0.01" mass="0.5" />

File: tbd_podi_description/urdf/podi.gazebo.xacro (robot description, xacro)
@@ -12,4 +12,5 @@
       <publishWheelJointState>true</publishWheelJointState>
       <publishWheelTF>false</publishWheelTF>
+      <publishOdom>true</publishOdom>
       <wheelAcceleration>1</wheelAcceleration>
       <commandTopic>/RosAria/cmd_vel</commandTopic> <!-- We choose to name it to match the robot's IRL command name-->
@@ -17,5 +18,5 @@
       <odometryFrame>$(arg robot_name)_odom</odometryFrame>
       <robotBaseFrame>$(arg robot_name)_base_link</robotBaseFrame>
-      <odometrySource>encoder</odometrySource>      <!-- The options are world and encoder. World means getting it straight from Gazebo -->
+      <odometrySource>world</odometrySource>      <!-- The options are world and encoder. World means getting it straight from Gazebo -->
       <!-- Zhi (2021-04-12) We use the world instead of encoder because the odometry is so much more worse in simulation for some reason.
       When Podi turns, the whole laser map is moved by nearly 45 degrees which is unrealistics. If you can figure out the difference. Dropping
