Commit message: Added Azure Kinect

File: tbd_podi_description/urdf/podi.gazebo.xacro (robot description, xacro)
@@ -67,6 +67,6 @@
     <visual>
       <plugin name="screen_video_controller" filename="libgazebo_ros_video.so">
-        <height>1080</height>
-        <width>1920</width>
+        <height>1280</height>
+        <width>720</width>
         <topicName>screen_face</topicName>
         <robotNamespace>${robotname}</robotNamespace>
@@ -74,38 +74,20 @@
     </visual>
   </gazebo>
-  <gazebo reference="${robotname}_front_camera">
-    <sensor type="camera" name="front_camera">
+  <gazebo reference="camera_base">
+    <sensor type="depth" name="front_depth_camera">
       <update_rate>30.0</update_rate>
-      <camera name="head">
+      <camera name="front_camera">
         <horizontal_fov>1.57079632679</horizontal_fov>
         <image>
-          <width>2560</width>
-          <height>720</height>
+          <width>1920</width>
+          <height>1080</height>
           <format>R8G8B8</format>
         </image>
-        <clip>
-          <near>0.02</near>
-          <far>300</far>
-        </clip>
-        <noise>
-          <type>gaussian</type>
-          <mean>0.0</mean>
-          <stddev>0.007</stddev>
-        </noise>
       </camera>
-      <plugin name="camera_controller" filename="libgazebo_ros_camera.so">
-        <alwaysOn>true</alwaysOn>
-        <updateRate>0.0</updateRate>
-        <cameraName>front_camera</cameraName>
-        <imageTopicName>image_raw</imageTopicName>
-        <cameraInfoTopicName>camera_info</cameraInfoTopicName>
-        <frameName>${robotname}_front_camera</frameName>
+      <plugin name="head_depth_camera" filename="libgazebo_ros_depth_camera.so">
+        <cameraName>azure_kinect</cameraName>
+        <frameName>camera_point</frameName>
         <robotNamespace>${robotname}</robotNamespace>
-        <hackBaseline>0.07</hackBaseline>
-        <distortionK1>0.0</distortionK1>
-        <distortionK2>0.0</distortionK2>
-        <distortionK3>0.0</distortionK3>
-        <distortionT1>0.0</distortionT1>
-        <distortionT2>0.0</distortionT2>
+        <pointCloudCutoff>2.0</pointCloudCutoff>
       </plugin>
     </sensor>

File: tbd_podi_description/urdf/podi.urdf.xacro (robot description, xacro)
@@ -3,6 +3,7 @@
     xmlns:xacro="http://ros.org/wiki/xacro">
     <xacro:property name="robotname" value="podi" />
-    <!-- Inport inertia functions -->
+    <!-- Inport helper functions -->
     <xacro:include filename="$(find tbd_podi_description)/urdf/inertia_tensors.xacro"/>
+    <xacro:include filename="$(find tbd_podi_description)/urdf/azure_kinect.urdf.xacro"/>
     <!-- Import the base robot -->
     <xacro:include filename="$(find tbd_podi_description)/urdf/pioneer3dx.urdf.xacro"/>

File: tbd_podi_description/urdf/podi_structure.xacro (robot description, xacro)
@@ -92,31 +92,18 @@
         <child link="${robotname}_display"/>
     </joint>
-    <link name="${robotname}_front_camera">
+    <link name="${robotname}_camera_mount">
         <inertial>
-            <mass value="0.01" />
+            <mass value="0.0001" />
             <origin xyz="0 0 0" />
             <inertia ixx="1" ixy="0" ixz="0" iyy="1" iyz="0" izz="1" />
         </inertial>
-        <visual>
-            <origin xyz="0 0 0" rpy="0 0 0"/>
-            <geometry name="zed">
-                <mesh filename="package://tbd_podi_description/meshes/zed.stl"/>
-            </geometry>
-            <material name="laser_scanner_color">
-                <color rgba="1 1 1 1"/>
-            </material>
-        </visual>
-        <collision>
-            <origin xyz="0 0 0" rpy="0 0 0"/>
-            <geometry name="zed">
-                <mesh filename="package://tbd_podi_description/meshes/zed.stl"/>
-            </geometry>
-        </collision>
     </link>
-   <joint name="camera_to_screen_joint" type="fixed">
-        <origin xyz="0 0 ${face_screen_height/2 + 0.025}" rpy="0 0 0"/>
+   <joint name="camera_mount_to_screen_joint" type="fixed">
+        <origin xyz="0.025 0 ${face_screen_height/2 + 0.025}" rpy="0 0 0"/>
         <axis xyz="0 1 0"/>
         <parent link="${robotname}_face_screen"/>
-        <child link="${robotname}_front_camera"/>
+        <child link="${robotname}_camera_mount"/>
     </joint>
+    <!-- Include Azure Kinect -->
+    <xacro:insert_azure_kinect parent="${robotname}_camera_mount" tf_prefix=""/>
 </robot>

Commit message: add ZED2

File: tbd_podi_description/urdf/podi.gazebo.xacro (robot description, xacro)
@@ -64,5 +64,5 @@
     </sensor>
   </gazebo>
-  <gazebo reference="${robotname}_display">
+  <gazebo reference="display">
     <visual>
       <plugin name="screen_video_controller" filename="libgazebo_ros_video.so">
@@ -74,5 +74,5 @@
     </visual>
   </gazebo>
-  <gazebo reference="camera_base">
+  <gazebo reference="zed_left_camera_optical_frame">
     <sensor type="depth" name="front_depth_camera">
       <update_rate>30.0</update_rate>
@@ -86,6 +86,6 @@
       </camera>
       <plugin name="head_depth_camera" filename="libgazebo_ros_depth_camera.so">
-        <cameraName>azure_kinect</cameraName>
-        <frameName>camera_point</frameName>
+        <cameraName>front_camera</cameraName>
+        <frameName>${robotname}/zed_left_camera_optical_frame</frameName>
         <robotNamespace>${robotname}</robotNamespace>
         <pointCloudCutoff>2.0</pointCloudCutoff>
@@ -93,5 +93,5 @@
     </sensor>
   </gazebo>
-  <gazebo reference="camera_base">
+  <!-- <gazebo reference="zed_left_camera_optical_frame">
     <gravity>true</gravity>
     <sensor type="imu_sensor" name="azure_imu">
@@ -112,4 +112,4 @@
       <pose>0 0 0 0 0 0</pose>
     </sensor>
-  </gazebo>
+  </gazebo> -->
 </robot>

File: tbd_podi_description/urdf/podi_structure.xacro (robot description, xacro)
@@ -27,5 +27,5 @@
     <xacro:property name="face_screen_height" value="0.2373" />
     <xacro:property name="face_screen_length" value="0.169" />
-    <link name="${robotname}_face_screen">
+    <link name="face_screen">
         <xacro:box_inertial x="${face_screen_width}" y="${face_screen_length}" z="${face_screen_height}" mass="0.429" />
         <visual>
@@ -55,5 +55,5 @@
         <origin xyz="0 0 0" rpy="0 0 0"/>
         <parent link="head"/>
-        <child link="${robotname}_face_screen"/>
+        <child link="face_screen"/>
     </joint>
     <joint name="screen_to_laser_scanner_joint" type="fixed">
@@ -65,5 +65,5 @@
     <xacro:property name="display_height" value="0.10125" />
     <xacro:property name="display_length" value="0.18" />
-    <link name="${robotname}_display">
+    <link name="display">
         <inertial>
             <mass value="0.01" />
@@ -76,5 +76,5 @@
                 <box size=" ${display_length} ${display_height} ${display_width}" />
             </geometry>
-            <material name="${robotname}_display_color">
+            <material name="$display_color">
                 <color rgba="0 0 0 1"/>
             </material>
@@ -89,8 +89,21 @@
     <joint name="display_to_screen_joint" type="fixed">
         <origin xyz="0.01 0 0" rpy="${3.1415927/2.0} 0 ${3.1415927/2.0}"/>
-        <parent link="${robotname}_face_screen"/>
-        <child link="${robotname}_display"/>
+        <parent link="face_screen"/>
+        <child link="display"/>
     </joint>
-    <link name="${robotname}_camera_mount">
+   <joint name="camera_mount_to_screen_joint" type="fixed">
+        <origin xyz="0.025 0 ${face_screen_height/2 + 0.025}" rpy="0 0 0"/>
+        <axis xyz="0 1 0"/>
+        <parent link="face_screen"/>
+        <child link="front_camera_mount"/>
+    </joint>
+    <xacro:arg name="base_frame" default="front_camera_mount"/>
+    <xacro:arg name="camera_model" default="zed2"/>
+    <xacro:include filename="$(find tbd_podi_description)/urdf/zed_descr.urdf.xacro">
+    </xacro:include>
+    <!-- camera_name="zed2" camera_model="zed2" base_frame="${robotname_camera_mount}"/> -->
+    <!-- Include Azure Kinect -->
+    <!-- <xacro:insert_azure_kinect parent="front_camera_mount" tf_prefix=""/> -->
+    <!-- <link name="front_camera_mount">
         <inertial>
             <mass value="0.0001" />
@@ -99,11 +112,4 @@
         </inertial>
     </link>
-   <joint name="camera_mount_to_screen_joint" type="fixed">
-        <origin xyz="0.025 0 ${face_screen_height/2 + 0.025}" rpy="0 0 0"/>
-        <axis xyz="0 1 0"/>
-        <parent link="${robotname}_face_screen"/>
-        <child link="${robotname}_camera_mount"/>
-    </joint>
-    <!-- Include Azure Kinect -->
-    <xacro:insert_azure_kinect parent="${robotname}_camera_mount" tf_prefix=""/>
+     -->
 </robot>

File: tbd_podi_description/urdf/zed_descr.urdf.xacro (robot description, xacro)
@@ -16,9 +16,18 @@
 -->
 <robot name="stereolabs_camera" xmlns:xacro="http://ros.org/wiki/xacro">
-<!-- Includes -->
-    <xacro:include filename="$(find zed_wrapper)/urdf/include/materials.urdf.xacro" />
+    <!-- Includes -->
+    <material name="zed_mat">
+        <color rgba="0.8 0.8 0.8 0.8"/>
+    </material>
+    <material name="zedm_mat">
+        <color rgba="0 0 0 0.9"/>
+    </material>
+    <material name="zed2_mat">
+        <color rgba="0.25 0.25 0.25 0.99"/>
+    </material>
     <!-- Arguments -->
     <xacro:arg name="camera_name"   default="zed" />
     <xacro:arg name="camera_model"  default="zed" />
+    <xacro:arg name="base_frame"    default="base_link" />
     <xacro:arg name="cam_pos_x"     default="0.0" />
     <xacro:arg name="cam_pos_y"     default="0.0" />
@@ -40,8 +49,8 @@
     </xacro:if>
 <!-- base_link -->
-    <link name="$(arg camera_name)_base_link" />
+    <link name="$(arg base_frame)" />
 <!-- Camera Center -->
     <joint name="$(arg camera_name)_camera_center_joint" type="fixed">
-        <parent link="$(arg camera_name)_base_link"/>
+        <parent link="$(arg base_frame)"/>
         <child link="$(arg camera_name)_camera_center"/>
         <origin xyz="$(arg cam_pos_x) $(arg cam_pos_y) $(arg cam_pos_z)" rpy="$(arg cam_roll) $(arg cam_pitch) $(arg cam_yaw)" />
@@ -51,5 +60,5 @@
             <origin xyz="0 0 0" rpy="0 0 0"/>
             <geometry>
-                <mesh filename="package://zed_wrapper/urdf/models/${model}.stl" />
+                <mesh filename="package://tbd_podi_description/meshes/${model}.stl" />
             </geometry>
             <material name="${model}_mat" />
@@ -82,3 +91,30 @@
     </joint>
     <link name="$(arg camera_name)_right_camera_optical_frame"/>
+<!-- ZED2 Sensors -->
+    <xacro:if value="${model == 'zed2'}">
+        <joint name="$(arg camera_name)_mag_joint" type="fixed">
+            <parent link="$(arg camera_name)_camera_center"/>
+            <child link="$(arg camera_name)_mag_link"/>
+            <origin xyz="0 0 0" rpy="0 0 0" />
+        </joint>
+        <link name="$(arg camera_name)_mag_link" />
+        <joint name="$(arg camera_name)_baro_joint" type="fixed">
+            <parent link="$(arg camera_name)_camera_center"/>
+            <child link="$(arg camera_name)_baro_link"/>
+            <origin xyz="0 0 0" rpy="0 0 0" />
+        </joint>
+        <link name="$(arg camera_name)_baro_link" />
+        <joint name="$(arg camera_name)_temp_left_joint" type="fixed">
+            <parent link="$(arg camera_name)_left_camera_frame"/>
+            <child link="$(arg camera_name)_temp_left_link"/>
+            <origin xyz="0 0 0" rpy="0 0 0" />
+        </joint>
+        <link name="$(arg camera_name)_temp_left_link" />
+        <joint name="$(arg camera_name)_temp_right_joint" type="fixed">
+            <parent link="$(arg camera_name)_right_camera_frame"/>
+            <child link="$(arg camera_name)_temp_right_link"/>
+            <origin xyz="0 0 0" rpy="0 0 0" />
+        </joint>
+        <link name="$(arg camera_name)_temp_right_link" />
+    </xacro:if>
 </robot>

Commit message: 1.3.0 - Better URDF

File: tbd_podi_description/urdf/podi.gazebo.xacro (robot description, xacro)
@@ -74,5 +74,5 @@
     </visual>
   </gazebo>
-  <gazebo reference="zed_left_camera_optical_frame">
+  <gazebo reference="zed_left_camera_frame">
     <sensor type="depth" name="front_depth_camera">
       <update_rate>30.0</update_rate>
@@ -93,5 +93,5 @@
     </sensor>
   </gazebo>
-  <!-- <gazebo reference="zed_left_camera_optical_frame">
+  <!-- <gazebo reference="zed_left_camera_frame">
     <gravity>true</gravity>
     <sensor type="imu_sensor" name="azure_imu">

File: tbd_podi_description/urdf/podi.urdf.xacro (robot description, xacro)
@@ -3,4 +3,6 @@
     xmlns:xacro="http://ros.org/wiki/xacro">
     <xacro:property name="robotname" value="podi" />
+    <!-- "fixed" if you don't want the handle to move. "move" for full rotation -->
+    <xacro:property name="handle_control" value="fixed" />
     <!-- Inport helper functions -->
     <xacro:include filename="$(find tbd_podi_description)/urdf/inertia_tensors.xacro"/>

File: tbd_podi_description/urdf/podi_handle.xacro (robot description, xacro)
@@ -113,5 +113,10 @@
         <parent link="handle_base"/>
         <child link="handle_bottom_plate"/>
-        <limit lower="-1.57" upper="1.57" effort="1" velocity="1" />
+        <xacro:if value="${handle_control == 'fixed'}">
+            <limit lower="-0.01" upper="0.01" effort="1" velocity="1" />
+        </xacro:if>
+        <xacro:if value="${handle_control == 'move'}">
+            <limit lower="-1.57" upper="1.57" effort="1" velocity="1" />
+        </xacro:if>
     </joint>
     <joint name="handle_bottom_plate_to_back_plate" type="fixed">

Commit message: new launch files

File: tbd_podi_description/urdf/podi.gazebo.xacro (robot description, xacro)
@@ -13,4 +13,7 @@
       <publishWheelTF>false</publishWheelTF>
       <publishOdom>true</publishOdom>
+      <publishOdomTF>false</publishOdomTF>
+      <publishTf>true</publishTf>
+      <rosDebugLevel>na</rosDebugLevel>
       <wheelAcceleration>1</wheelAcceleration>
       <commandTopic>/RosAria/cmd_vel</commandTopic> <!-- We choose to name it to match the robot's IRL command name-->

File: tbd_podi_description/urdf/podi_structure.xacro (robot description, xacro)
@@ -9,4 +9,24 @@
     <xacro:property name="display_height" value="0.147" />
     <xacro:property name="display_length" value="0.197" />
+    <link name="$(arg robot_name)_uwb">
+    	<xacro:box_inertial x="0.01" y="0.01" z="0.01" mass="0.1" />
+    	<visual>
+    		<origin xyz="0 0 0" rpy="0 0 0"/>
+    		<geometry>
+                	<box size="0.01 0.01 0.01" />
+            	</geometry>
+        </visual>
+        <collision>
+            <origin xyz="0 0 0" rpy="0 0 0"/>
+            <geometry>
+                <box size="0.01 0.01 0.01" />
+            </geometry>
+        </collision>
+    </link>
+    <joint name="$(arg robot_name)_base_to_uwb" type="fixed">
+        <origin xyz="0 0 1.054" rpy="0 0 0"/>
+        <parent link="$(arg robot_name)_base_link"/>
+        <child link="$(arg robot_name)_uwb"/>
+    </joint>
     <link name="$(arg robot_name)_laser_scanner">
         <xacro:box_inertial x="0.105" y="0.102" z="0.152" mass="0.429" />
